Commit message: Claude full implementation

File: ros2_ws/src/my_robot_description/urdf/camera.urdf.xacro (robot description, xacro)
@@ -53,6 +53,7 @@
         <parent link="base_link"/>
         <child link="camera_link"/>
-        <!-- Keep the existing camera mounting position. -->
-        <origin xyz="0.15 0 0.10" rpy="0 0 0"/>
+        <!-- Mounting bracket was rotated 180 deg about the camera's own
+             boresight (+X, forward), flipping the sensor upside-down. -->
+        <origin xyz="0.15 0 0.10" rpy="3.14159265359 0 0"/>
     </joint>
     <!-- ROS optical convention: +Z forward, +X right, +Y down. -->
